File: mumble.sch (KiCad schematic (older format))
At the start: 76 parts, among them J1 Serial, J10 M1, J11 X_MOT, J12 M0, J13 M1, J14 M0, J15 M1, J16 Z_MOT, J17 Y_MOT, J2 Servo, J3 VM sel, J4 BATT, J5 Charge, J6 Limit Switches, J7 Front Panel, J8 Machine Functions, J9 M0, Q1 IRLML9301, Q2 IRLML9301, SW1 SW_SPST, SW2 Reset, SW3 Hold Button, SW4 Start Button, SW5 Abort Button, SW6 Program, U1 TP4054, U2 ESP32-WROOM, U3 AP2204K-3.3, U4 DRV8834, U5 DRV8834, U6 DRV8834

Commit message: Routed PCB
Parts:
- removed J4: BATT, Connectors_Terminal_Blocks:TerminalBlock_bornier-2_P5.08mm, symbol mumble-rescue:Conn_01x02
- removed J5: Charge, Connectors_Terminal_Blocks:TerminalBlock_bornier-2_P5.08mm, symbol mumble-rescue:Conn_01x02
- added BT101: Battery, Connectors_JST:JST_EH_B02B-EH-A_02x2.50mm_Straight, symbol device:Battery
- added D101: LED, LEDs:LED_0805, symbol device:LED
- added J101: USB_B_Micro, Connectors_USB:USB_Micro-B_Wuerth-629105150521, symbol Connector:USB_B_Micro
- added R101: 330, Resistors_SMD:R_0805_HandSoldering, symbol device:R
- J1: footprint (none) -> Pin_Headers:Pin_Header_Straight_1x06_Pitch2.54mm
- J11, J16, J17: footprint (none) -> Pin_Headers:Pin_Header_Straight_1x04_Pitch2.54mm
- J6, J7: footprint (none) -> Pin_Headers:Pin_Header_Straight_2x04_Pitch2.54mm
- J8: footprint (none) -> Pin_Headers:Pin_Header_Straight_2x06_Pitch2.54mm
- RV1, RV2, RV3: footprint (none) -> Potentiometers:Potentiometer_Trimmer-EVM3E
- SW1: footprint (none) -> Accelerando:TorchButton
- SW2, SW3, SW4, SW5, SW6: footprint Buttons_Switches_THT:SW_PUSH_6mm_h4.3mm -> Accelerando:TVBM02
- U2: footprint ESP32-footprints-Lib:ESP32-WROOM -> ESP32:ESP32-WROOM
- U4, U5, U6: footprint (none) -> Accelerando:HTSSOP-24
Connections:
- net labels added: +3V3
- wire segments 416 -> 419

Commit message: Updated caps and sense resistors
Parts:
- C10, C18, C19: footprint Capacitors_SMD:C_0805_HandSoldering -> Capacitors_THT:CP_Radial_D5.0mm_P2.50mm
- R12, R13, R18, R19, R20, R21: footprint Resistors_SMD:R_0805_HandSoldering -> Resistors_SMD:R_1206
Changed lines of the file:
@@
 F 0 "R12" V 9980 7570 50  0000 L CNN
 F 1 "0.1R" H 9980 7510 50  0000 L CNN
-F 2 "Resistors_SMD:R_0805_HandSoldering" H 9950 7550 50  0001 C CNN
+F 2 "Resistors_SMD:R_1206" H 9950 7550 50  0001 C CNN
 F 3 "" H 9950 7550 50  0001 C CNN
 	1    9950 7550
@@
 F 0 "R13" V 9980 8470 50  0000 L CNN
 F 1 "0.1R" H 9980 8410 50  0000 L CNN
-F 2 "Resistors_SMD:R_0805_HandSoldering" H 9950 8450 50  0001 C CNN
+F 2 "Resistors_SMD:R_1206" H 9950 8450 50  0001 C CNN
 F 3 "" H 9950 8450 50  0001 C CNN
 	1    9950 8450
@@
 F 0 "R20" V 14080 7570 50  0000 L CNN
 F 1 "0.1R" H 14080 7510 50  0000 L CNN
-F 2 "Resistors_SMD:R_0805_HandSoldering" H 14050 7550 50  0001 C CNN
+F 2 "Resistors_SMD:R_1206" H 14050 7550 50  0001 C CNN
 F 3 "" H 14050 7550 50  0001 C CNN
 	1    14050 7550
@@
 F 0 "R21" V 14080 8470 50  0000 L CNN
 F 1 "0.1R" H 14080 8410 50  0000 L CNN
-F 2 "Resistors_SMD:R_0805_HandSoldering" H 14050 8450 50  0001 C CNN
+F 2 "Resistors_SMD:R_1206" H 14050 8450 50  0001 C CNN
 F 3 "" H 14050 8450 50  0001 C CNN
 	1    14050 8450
@@
 F 0 "R18" V 14080 3020 50  0000 L CNN
 F 1 "0.1R" H 14080 2960 50  0000 L CNN
-F 2 "Resistors_SMD:R_0805_HandSoldering" H 14050 3000 50  0001 C CNN
+F 2 "Resistors_SMD:R_1206" H 14050 3000 50  0001 C CNN
 F 3 "" H 14050 3000 50  0001 C CNN
 	1    14050 3000
@@
 F 0 "R19" V 14080 3920 50  0000 L CNN
 F 1 "0.1R" H 14080 3860 50  0000 L CNN
-F 2 "Resistors_SMD:R_0805_HandSoldering" H 14050 3900 50  0001 C CNN
+F 2 "Resistors_SMD:R_1206" H 14050 3900 50  0001 C CNN
 F 3 "" H 14050 3900 50  0001 C CNN
 	1    14050 3900
@@
 F 0 "C18" H 13560 1470 50  0000 L CNN
 F 1 "100uF" H 13560 1320 50  0000 L CNN
-F 2 "Capacitors_SMD:C_0805_HandSoldering" H 13550 1400 50  0001 C CNN
+F 2 "Capacitors_THT:CP_Radial_D5.0mm_P2.50mm" H 13550 1400 50  0001 C CNN
 F 3 "" H 13550 1400 50  0001 C CNN
 	1    13550 1400
@@
 F 0 "C19" H 13660 6020 50  0000 L CNN
 F 1 "100uF" H 13660 5870 50  0000 L CNN
-F 2 "Capacitors_SMD:C_0805_HandSoldering" H 13650 5950 50  0001 C CNN
+F 2 "Capacitors_THT:CP_Radial_D5.0mm_P2.50mm" H 13650 5950 50  0001 C CNN
 F 3 "" H 13650 5950 50  0001 C CNN
 	1    13650 5950
@@
 F 0 "C10" H 9510 6020 50  0000 L CNN
 F 1 "100uF" H 9510 5870 50  0000 L CNN
-F 2 "Capacitors_SMD:C_0805_HandSoldering" H 9500 5950 50  0001 C CNN
+F 2 "Capacitors_THT:CP_Radial_D5.0mm_P2.50mm" H 9500 5950 50  0001 C CNN
 F 3 "" H 9500 5950 50  0001 C CNN
 	1    9500 5950
