File: mumble.sch (KiCad schematic (older format))
At the start: 80 parts, among them J1 Serial, J10 M1, J101 USB_B_Micro, J11 X_MOT, J12 M0, J13 M1, J14 M0, J15 M1, J16 Z_MOT, J17 Y_MOT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

Commit message: Updated power button and USB connector
Parts:
- J101: footprint Connectors_USB:USB_Micro-B_Wuerth-629105150521 -> Accelerando:USB_Micro
- gave numbers to parts that had none: 2
Changed lines of the file:
@@
 F 0 "J101" V 2409 1079 50  0000 L CNN
 F 1 "USB_B_Micro" V 2500 1079 50  0000 L CNN
-F 2 "Connectors_USB:USB_Micro-B_Wuerth-629105150521" H 2550 700 50  0001 C CNN
+F 2 "Accelerando:USB_Micro" H 2550 700 50  0001 C CNN
 F 3 "~" H 2550 700 50  0001 C CNN
 	1    2400 750
@@
 VBAT
 $Comp
-L device:LED D?
+L device:LED D102
 U 1 1 5B7C7782
 P 8600 4050
-F 0 "D?" V 8638 3933 50  0000 R CNN
+F 0 "D102" V 8638 3933 50  0000 R CNN
 F 1 "LED" V 8547 3933 50  0000 R CNN
 F 2 "LEDs:LED_0805" H 8600 4050 50  0001 C CNN
@@
 $EndComp
 $Comp
-L device:R R?
+L device:R R102
 U 1 1 5B7C7788
 P 8600 4350
-F 0 "R?" H 8670 4396 50  0000 L CNN
+F 0 "R102" H 8670 4396 50  0000 L CNN
 F 1 "330" H 8670 4305 50  0000 L CNN
 F 2 "Resistors_SMD:R_0805_HandSoldering" V 8530 4350 50  0001 C CNN
@@
 $EndComp
 $Comp
-L mumble-rescue:GND #PWR?
+L mumble-rescue:GND #PWR0105
 U 1 1 5B7C778E
 P 8600 4500
-F 0 "#PWR?" H 8600 4250 50  0001 C CNN
+F 0 "#PWR0105" H 8600 4250 50  0001 C CNN
 F 1 "GND" H 8600 4350 50  0000 C CNN
 F 2 "" H 8600 4500 50  0001 C CNN

Commit message: Saved
Parts:
- SW1: footprint Accelerando:TorchButton -> Accelerando:CherryPowerSwitch
Changed lines of the file:
@@
 F 0 "SW1" H 1750 1835 50  0000 C CNN
 F 1 "SW_SPST" H 1750 1744 50  0000 C CNN
-F 2 "Accelerando:TorchButton" H 1750 1600 50  0001 C CNN
+F 2 "Accelerando:CherryPowerSwitch" H 1750 1600 50  0001 C CNN
 F 3 "" H 1750 1600 50  0001 C CNN
 	1    1750 1600

Commit message: Updated to V1.2 of PCB
Parts:
- removed C13: 4.7uF, Capacitors_SMD:C_0805_HandSoldering, symbol mumble-rescue:C_Small
- removed C15: 10uF, Capacitors_SMD:C_0805_HandSoldering, symbol mumble-rescue:CP_Small
- removed C17: 2.2uF, Capacitors_SMD:C_0805_HandSoldering, symbol mumble-rescue:C_Small
- removed C19: 100uF, Capacitors_THT:CP_Radial_D5.0mm_P2.50mm, symbol mumble-rescue:CP_Small
- removed C21: 0.01uF, Capacitors_SMD:C_0805_HandSoldering, symbol mumble-rescue:C_Small
- removed J10, J13, J15: M1, Pin_Headers:Pin_Header_Straight_1x03_Pitch2.54mm, symbol mumble-rescue:Conn_01x03
- removed J12, J14, J9: M0, Pin_Headers:Pin_Header_Straight_1x03_Pitch2.54mm, symbol mumble-rescue:Conn_01x03
- removed J17: Y_MOT, Pin_Headers:Pin_Header_Straight_1x04_Pitch2.54mm, symbol Connector:Conn_01x04
- removed J6: Limit Switches, Pin_Headers:Pin_Header_Straight_2x04_Pitch2.54mm, symbol Connector:Conn_02x04_Odd_Even
- removed J7: Front Panel, Pin_Headers:Pin_Header_Straight_2x04_Pitch2.54mm, symbol Connector:Conn_02x04_Odd_Even
- removed J8: Machine Functions, Pin_Headers:Pin_Header_Straight_2x06_Pitch2.54mm, symbol Connector:Conn_02x06_Odd_Even
- removed R15, R17: 47k, Resistors_SMD:R_0805_HandSoldering, symbol mumble-rescue:R_Small
- removed R20, R21: 0.1R, Resistors_SMD:R_1206, symbol mumble-rescue:R_Small
- removed RV3: 10k, Potentiometers:Potentiometer_Trimmer-EVM3E, symbol device:POT_TRIM
- removed U6: DRV8834, Accelerando:HTSSOP-24, symbol mumble-rescue:DRV8834-Accelerando
- added D103: CHRG, LEDs:LED_0805, symbol device:LED
- added JP101, JP102, JP103, JP104: Jumper_3_Bridged12, Jumper:SolderJumper-3_P1.3mm_Bridged2Bar12_Pad1.0x1.5mm, symbol Jumper:Jumper_3_Bridged12
- added R103: 330, Resistors_SMD:R_0805_HandSoldering, symbol device:R
- U4, U5: symbol mumble-rescue:DRV8834-Accelerando -> Accelerando:DRV8834
Connections:
- net labels added: BATT_PROT, BATT_SWITCHED, VCP_X, VCP_Y, VINT_X, VINT_Y
- net labels removed: VBAT, VCC, VCP, VINT
- wire segments 418 -> 262
- no-connect marks 4 -> 3
Other:
- note added: "NB: SURFACE MOUNT THIS"
- moved on the sheet: C12, C14, C16, C18, C20, Q1, R14, R16, R18, R19, SW1, SW3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

Commit message: version 1.3, fixed nsleep, chrg led not working. change motor pinout for neater routing.
Parts:
- added R104, R105: 47k, Resistor_SMD:R_0805_2012Metric, symbol mumble-rescue:R_Small
- BT101: symbol device:Battery -> Device:Battery
- D101, D102, D103: footprint LEDs:LED_0805 -> LED_SMD:LED_0805_2012Metric; symbol device:LED -> Device:LED
- J1: footprint Pin_Headers:Pin_Header_Straight_1x06_Pitch2.54mm -> Connector_PinHeader_2.54mm:PinHeader_1x06_P2.54mm_Vertical; symbol Connector:Conn_01x06 -> Connector_Generic:Conn_01x06
- J11, J16: symbol Connector:Conn_01x04 -> Connector_Generic:Conn_01x04
- R101, R102, R103: symbol device:R -> Device:R
- RV1, RV2: symbol device:POT_TRIM -> Device:R_POT_TRIM
Connections:
- wire segments 262 -> 264
Changed lines of the file:
@@
 Connection ~ 5500 8050
 $Comp
-L Connector:Conn_01x06 J1
+L Connector_Generic:Conn_01x06 J1
 U 1 1 5B74C30C
 P 1800 2800
 F 0 "J1" H 1720 3217 50  0000 C CNN
 F 1 "Serial" H 1720 3126 50  0000 C CNN
-F 2 "Pin_Headers:Pin_Header_Straight_1x06_Pitch2.54mm" H 1800 2800 50  0001 C CNN
+F 2 "Connector_PinHeader_2.54mm:PinHeader_1x06_P2.54mm_Vertical" H 1800 2800 50  0001 C CNN
 F 3 "~" H 1800 2800 50  0001 C CNN
 	1    1800 2800
@@
 	4000 4000 4450 4000
 $Comp
-L Connector:Conn_01x04 J11
+L Connector_Generic:Conn_01x04 J11
 U 1 1 5BA199BE
 P 10300 7100
@@
 	9950 8300 9950 8350
 Wire Wire Line
-	10100 7100 9900 7100
-Wire Wire Line
-	9900 7850 10050 7850
-Wire Wire Line
 	10050 7850 10050 7200
 Wire Wire Line
@@
 Wire Wire Line
 	10100 7300 10100 8100
-Wire Wire Line
-	10100 8100 9900 8100
-Wire Wire Line
-	9900 7100 9900 7200
 Wire Wire Line
 	9200 8850 9200 8950
@@
 	8450 8450 8450 8550
 Connection ~ 8450 8550
-Wire Wire Line
-	9900 7000 10100 7000
 Connection ~ 9200 8850
 Wire Wire Line
@@
 $EndComp
 $Comp
-L device:POT_TRIM RV1
+L Device:R_POT_TRIM RV1
 U 1 1 5BA19A68
 P 8800 8950
@@
 Y_DIR
 $Comp
-L Connector:Conn_01x04 J16
+L Connector_Generic:Conn_01x04 J16
 U 1 1 5B821997
 P 14500 7100
@@
 $EndComp
 $Comp
-L device:POT_TRIM RV2
+L Device:R_POT_TRIM RV2
 U 1 1 5B821A3C
 P 13000 8950
@@
 	2300 1050 2400 1050
 $Comp
-L device:Battery BT101
+L Device:Battery BT101
 U 1 1 5B7597E1
 P 1950 1800
@@
 $EndComp
 $Comp
-L device:LED D101
+L Device:LED D101
 U 1 1 5B78A65D
 P 5800 3400
 F 0 "D101" V 5838 3283 50  0000 R CNN
 F 1 "LED" V 5747 3283 50  0000 R CNN
-F 2 "LEDs:LED_0805" H 5800 3400 50  0001 C CNN
+F 2 "LED_SMD:LED_0805_2012Metric" H 5800 3400 50  0001 C CNN
 F 3 "~" H 5800 3400 50  0001 C CNN
 	1    5800 3400
@@
 $EndComp
 $Comp
-L device:R R101
+L Device:R R101
 U 1 1 5B78A9C7
 P 5800 3700
@@
 $EndComp
 $Comp
-L device:LED D102
+L Device:LED D102
 U 1 1 5B7C7782
 P 6500 3400
 F 0 "D102" V 6538 3283 50  0000 R CNN
 F 1 "LED" V 6447 3283 50  0000 R CNN
-F 2 "LEDs:LED_0805" H 6500 3400 50  0001 C CNN
+F 2 "LED_SMD:LED_0805_2012Metric" H 6500 3400 50  0001 C CNN
 F 3 "~" H 6500 3400 50  0001 C CNN
 	1    6500 3400
@@
 $EndComp
 $Comp
-L device:R R102
+L Device:R R102
 U 1 1 5B7C7788
 P 6500 3700
@@
 Wire Wire Line
 	7500 7700 8050 7700
-Text Label 8500 7600 2    50   ~ 0
-VINT_X
 Wire Wire Line
 	11750 7200 12000 7200
@@
 Text Label 11300 7550 0    50   ~ 0
 VINT_Y
-Text Label 12700 7600 2    50   ~ 0
-VINT_Y
 $Comp
 L mumble-rescue:+BATT #PWR0110
@@
 	1    0    0    -1
 $EndComp
-Connection ~ 1950 1600
 Text Label 950  1600 2    50   ~ 0
 BATT_SWITCHED
 $Comp
-L device:LED D103
+L Device:LED D103
 U 1 1 5B8F6FBA
 P 8000 3400
 F 0 "D103" V 8038 3283 50  0000 R CNN
 F 1 "CHRG" V 7947 3283 50  0000 R CNN
-F 2 "LEDs:LED_0805" H 8000 3400 50  0001 C CNN
+F 2 "LED_SMD:LED_0805_2012Metric" H 8000 3400 50  0001 C CNN
 F 3 "~" H 8000 3400 50  0001 C CNN
 	1    8000 3400
@@
 $EndComp
 $Comp
-L device:R R103
+L Device:R R103
 U 1 1 5B8F6FC0
 P 8000 3700
@@
 Wire Wire Line
 	2600 1400 3050 1400
+Text Label 3450 1400 0    50   ~ 0
+BATT_PROT
+$Comp
+L mumble-rescue:R_Small R104
+U 1 1 5C14831B
+P 8200 7700
+F 0 "R104" V 8230 7720 50  0000 L CNN
+F 1 "47k" H 8230 7660 50  0000 L CNN
+F 2 "Resistor_SMD:R_0805_2012Metric" H 8200 7700 50  0001 C CNN
+F 3 "" H 8200 7700 50  0001 C CNN
+	1    8200 7700
+	1    0    0    -1
+$EndComp
+Wire Wire Line
+	8500 7600 8200 7600
+Text Label 8200 7800 0    50   ~ 0
+VM
+$Comp
+L mumble-rescue:R_Small R105
+U 1 1 5C16CE90
+P 12400 7700
+F 0 "R105" V 12430 7720 50  0000 L CNN
+F 1 "47k" H 12430 7660 50  0000 L CNN
+F 2 "Resistor_SMD:R_0805_2012Metric" H 12400 7700 50  0001 C CNN
+F 3 "" H 12400 7700 50  0001 C CNN
+	1    12400 7700
+	1    0    0    -1
+$EndComp
+Wire Wire Line
+	12700 7600 12400 7600
+Text Label 12400 7800 0    50   ~ 0
+VM
+Wire Wire Line
+	10100 8100 9900 8100
+Wire Wire Line
+	9900 7850 10050 7850
+Wire Wire Line
+	9900 7000 10100 7000
+Wire Wire Line
+	9900 7100 9900 7200
+Wire Wire Line
+	9900 7100 10100 7100
 $EndSCHEMATC
