File: _saved_mumble.sch (KiCad schematic (older format))
At the start: 80 parts, among them J1 Serial, J10 M1, J101 USB_B_Micro, J11 X_MOT, J12 M0, J13 M1, J14 M0, J15 M1, J16 Z_MOT, J17 Y_MOT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

Commit message: Updated some of the errata
Parts:
- gave numbers to parts that had none: 2
Changed lines of the file:
@@
 VBAT
 $Comp
-L device:LED D?
+L device:LED D102
 U 1 1 5B7C7782
 P 8600 4050
-F 0 "D?" V 8638 3933 50  0000 R CNN
+F 0 "D102" V 8638 3933 50  0000 R CNN
 F 1 "LED" V 8547 3933 50  0000 R CNN
 F 2 "LEDs:LED_0805" H 8600 4050 50  0001 C CNN
@@
 $EndComp
 $Comp
-L device:R R?
+L device:R R102
 U 1 1 5B7C7788
 P 8600 4350
-F 0 "R?" H 8670 4396 50  0000 L CNN
+F 0 "R102" H 8670 4396 50  0000 L CNN
 F 1 "330" H 8670 4305 50  0000 L CNN
 F 2 "Resistors_SMD:R_0805_HandSoldering" V 8530 4350 50  0001 C CNN
@@
 $EndComp
 $Comp
-L mumble-rescue:GND #PWR?
+L mumble-rescue:GND #PWR0105
 U 1 1 5B7C778E
 P 8600 4500
-F 0 "#PWR?" H 8600 4250 50  0001 C CNN
+F 0 "#PWR0105" H 8600 4250 50  0001 C CNN
 F 1 "GND" H 8600 4350 50  0000 C CNN
 F 2 "" H 8600 4500 50  0001 C CNN

Commit message: Actually saved the PCB this time
Parts:
- J101: footprint Connectors_USB:USB_Micro-B_Wuerth-629105150521 -> Accelerando:USB_Micro
- SW1: footprint Accelerando:TorchButton -> Accelerando:CherryPowerSwitch
Changed lines of the file:
@@
 F 0 "SW1" H 1750 1835 50  0000 C CNN
 F 1 "SW_SPST" H 1750 1744 50  0000 C CNN
-F 2 "Accelerando:TorchButton" H 1750 1600 50  0001 C CNN
+F 2 "Accelerando:CherryPowerSwitch" H 1750 1600 50  0001 C CNN
 F 3 "" H 1750 1600 50  0001 C CNN
 	1    1750 1600
@@
 F 0 "J101" V 2409 1079 50  0000 L CNN
 F 1 "USB_B_Micro" V 2500 1079 50  0000 L CNN
-F 2 "Connectors_USB:USB_Micro-B_Wuerth-629105150521" H 2550 700 50  0001 C CNN
+F 2 "Accelerando:USB_Micro" H 2550 700 50  0001 C CNN
 F 3 "~" H 2550 700 50  0001 C CNN
 	1    2400 750
